File: Hardware/PCB/Eagle/Qwiic_Adaptive_Switch_Single.brd (EAGLE design)
At the start: 41.9 x 30.5 mm, 13 parts, among them J2 J2, SW1 CUI_SJ1-3513, SW2 CUI_SJ1-3513

Commit message: Updated the design.
Parts:
- removed U$1, U$13: (no value), SparkFun-Aesthetics:OSHW-LOGO-S
- added U$2: MILADOR-LOGO-, milador:MILADOR_LOGO1
- J1: value (none) -> QWIIC_RIGHT_ANGLE; device SparkFun-Connectors:1X04_1MM_RA -> milador_SMD:CONNECTORS_JST04_1MM_RA
- J2, J3: device SparkFun-Connectors:1X04_NO_SILK -> milador:CONNECTORS_1X04_NO_SILK
- R1, R2: value (none) -> R-US_0204/7; device MMC Eagle:RESISTOR_0205/7 -> milador:0204/7
