File: Hardware/PCB/Eagle/Qwiic_Adaptive_Switch.sch (EAGLE design)
At the start: 11 parts, among them J2 J2, SW1 CUI_SJ1-3513, SW2 CUI_SJ1-3513

Commit message: Added Single and I2C BOM files
Parts:
- removed JP1, JP2: STAND-OFF, SparkFun-Hardware:STAND-OFF
- added ADR0, ADR1, INT, PWR: JUMPER-SMT_2_NC_TRACE_SILK, SparkFun-Jumpers:JUMPER-SMT_2_NC_TRACE_SILK
- added ADR2: JUMPER-SMT_2_NC_TRACE_NO-SILK, SparkFun-Jumpers:JUMPER-SMT_2_NC_TRACE_NO-SILK
- added C1: 0.1uF, SparkFun-Capacitors:0.1UF-0603-25V-(+80/-20%)
- added D1: RED, SparkFun-LED:LED-RED0603
- added H1, H2: STAND-OFF, SparkFun-Hardware:STAND-OFF
- added I2C: JUMPER-SMT_3_2-NC_TRACE_SILK, SparkFun-Jumpers:JUMPER-SMT_3_2-NC_TRACE_SILK
- added J4: (no value), SparkFun-Connectors:CONN_041X04_NO_SILK
- added J7: (no value), SparkFun-Connectors:CONN_01PTH_NO_SILK_YES_STOP
- added LOGO1: OSHW-LOGOMINI, SparkFun-Aesthetics:OSHW-LOGOMINI
- added R3, R4, R5: 2.2k, SparkFun-Resistors:2.2KOHM-0603-1/10W-1%
- added R6: 10k, SparkFun-Resistors:10KOHM-0603-1/10W-1%
- added R7: 1k, SparkFun-Resistors:1KOHM-0603-1/10W-1%
- added U1: TCA9534, SparkFun-IC-Conversion:TCA9534U
- J1: device SparkFun-Connectors:I2C_STANDARDQWIIC -> SparkFun-Connectors:CONN_041X04_NO_SILK
- J2: value J2 -> QWIIC; device SparkFun-Connectors:CONN_041X04_NO_SILK_NO_POP -> SparkFun-Connectors:QWIIC_CONNECTORJS-1MM; PROD_ID (none) -> CONN-13694
- J3: value (none) -> QWIIC; device SparkFun-Connectors:CONN_041X04_NO_SILK_NO_POP -> SparkFun-Connectors:QWIIC_CONNECTORJS-1MM; PROD_ID (none) -> CONN-13694
- JP3, JP4: device SparkFun-Hardware:STAND-OFF -> SparkFun:STAND-OFF
- R1, R2: value (none) -> 2.2k; device MMC Eagle:RESISTOR-US-0204/7 -> SparkFun-Resistors:2.2KOHM-0603-1/10W-1%
Connections:
- removed net SCL/SCK: J1.4, J2.1, R2.1, SW2.2
- removed net SDA/MOSI: J1.3, J2.2, R1.1, SW1.2
- new net !INT: J7.1, R6.1, U1.!INT
- new net ADR0: ADR0.1, R5.2, U1.A0
- new net ADR1: ADR1.1, R3.2, U1.A1
- new net ADR2: ADR2.1, R1.2, U1.A2
- new net N$1: INT.1, R6.2
- new net N$2: D1.A, R7.1
- new net N$3: PWR.1, R7.2
- new net P0: SW1.2, U1.P0
- new net P1: SW2.2, U1.P1
- new net P2: J4.3, U1.P2
- new net P3: J4.4, U1.P3
- new net SCL: J1.4, J2.4, J3.4, R4.1, U1.SCL
- new net SCL_PU1: I2C.1, R2.2
- new net SDA: J1.3, J2.3, J3.3, R2.1, U1.SDA
- new net SDA_PU1: I2C.3, R4.2
- net 3.3V: now also ADR0.2, ADR1.2, ADR2.2, C1.1, I2C.2, INT.2, J2.2, J3.2, J4.2, PWR.2, U1.VCC; no longer J2.3, J3.3, R1.2, R2.2
- net GND: now also C1.2, D1.C, J2.1, J3.1, J4.1, R1.1, R3.1, R5.1, U1.GND; no longer J2.4, J3.4
Other:
- note added: "0 0 0 0x20"
- note added: "0 0 1 0x21"
- note added: "0 1 0 0x22"
- note added: "0 1 1 0x23"
- note added: "0: Open 1: Closed"
- note added: "1 0 0 0x24"
- note added: "1 0 1 0x25"
- note added: "1 1 0 0x26"
- note added: "1 1 1 0x27 (default)"
- note added: "ADR2 ADR1 ADR0 Address"
- note added: "Address Selection Jumpers"
- note added: "Connections"
- note added: "Cut the !INT jumper to remove the interrupt pullup if there is another pullup on !INT."
- note added: "Cut the I2C Jumpers to remove these pullups from the I2C bus"
- note added: "Cut the PWR Jumper to disable the PWR LED"
- note added: "Developed By: Kevin Kuwata"
- note added: "I2C->GPIO (TCA9534)"
- note added: "Modified By: Milad Hajihassan"
- note added: "VCC: 1.65-5.5V"
- note added: "v10"
- note removed: "Milad Hajihassan"
- note removed: "V1.0"
- note removed: "github.com/milador/Qwiic-Adaptive-Switch"
- moved on the sheet: R1, R2, SW1, SW2

Commit message: Updated design
Parts:
- removed J7: (no value), SparkFun-Connectors:CONN_01PTH_NO_SILK_YES_STOP
- added J5: (no value), SparkFun-Connectors:CONN_041X04_NO_SILK
- added R8, R9: 2.2k, SparkFun-Resistors:2.2KOHM-0603-1/10W-1%
- added U$17: MILADOR-SWITCH-NAME-SW1, milador:MILADOR-SWITCH-NAME-SW1
- added U$18: MILADOR-SWITCH-NAME-SW2, milador:MILADOR-SWITCH-NAME-SW2
- added U$6: MILADOR-LOGO-, milador:MILADOR-LOGO-
- ADR2: value JUMPER-SMT_2_NC_TRACE_NO-SILK -> JUMPER-SMT_2_NC_TRACE_SILK; device SparkFun-Jumpers:JUMPER-SMT_2_NC_TRACE_NO-SILK -> SparkFun-Jumpers:JUMPER-SMT_2_NC_TRACE_SILK
- J1, J4: value (none) -> QWIIC; device SparkFun-Connectors:CONN_041X04_NO_SILK -> SparkFun-Connectors:QWIIC_CONNECTORJS-1MM; PROD_ID (none) -> CONN-13694
- J2: value QWIIC -> (none); device SparkFun-Connectors:QWIIC_CONNECTORJS-1MM -> SparkFun-Connectors:CONN_01PTH_NO_SILK_YES_STOP; PROD_ID CONN-13694 -> (none)
- J3: value QWIIC -> (none); device SparkFun-Connectors:QWIIC_CONNECTORJS-1MM -> SparkFun-Connectors:CONN_041X04_NO_SILK; PROD_ID CONN-13694 -> (none)
- R3: value 2.2k -> 10k; device SparkFun-Resistors:2.2KOHM-0603-1/10W-1% -> SparkFun-Resistors:10KOHM-0603-1/10W-1%
- R4: value 2.2k -> 1k; device SparkFun-Resistors:2.2KOHM-0603-1/10W-1% -> SparkFun-Resistors:1KOHM-0603-1/10W-1%
- R5: value 2.2k -> 10k
- R6: value 10k -> 10K; device SparkFun-Resistors:10KOHM-0603-1/10W-1% -> SparkFun-Resistors:2.2KOHM-0603-1/10W-1%
- R7: value 1k -> 2.2k; device SparkFun-Resistors:1KOHM-0603-1/10W-1% -> SparkFun-Resistors:2.2KOHM-0603-1/10W-1%
Connections:
- net !INT: now also J2.1, R3.1; no longer J7.1, R6.1
- net 3.3V: now also J5.2, R5.2, R6.2; no longer J2.2
- net ADR0: now also R9.2; no longer R5.2
- net ADR1: now also R8.2; no longer R3.2
- net ADR2: now also R7.2; no longer R1.2
- net GND: now also J5.1, R7.1, R8.1, R9.1; no longer J2.1, R1.1, R3.1, R5.1
- net N$1: now also R3.2; no longer R6.2
- net N$2: now also R4.1; no longer R7.1
- net N$3: now also R4.2; no longer R7.2
- net P0: now also R5.1
- net P1: now also R6.1
- net P2: now also J5.3; no longer J4.3
- net P3: now also J5.4; no longer J4.4
- net SCL: now also J4.4, R1.1; no longer J2.4, R4.1
- net SDA: now also J4.3; no longer J2.3
- net SDA_PU1: now also R1.2; no longer R4.2
Other:
- moved on the sheet: ADR2, R1, R3, R4, R5, R6, R7, SW1, SW2

Commit message: Updated the design.
Parts:
- removed LOGO1: OSHW-LOGOMINI, SparkFun-Aesthetics:OSHW-LOGOMINI
- ADR0, ADR1, ADR2, INT, PWR: value JUMPER-SMT_2_NC_TRACE_SILK -> JUMPERS-SMT_2_NC_TRACE_SILK; device SparkFun-Jumpers:JUMPER-SMT_2_NC_TRACE_SILK -> milador_SMD:JUMPERS-SMT_2_NC_TRACE_SILK
- C1: device SparkFun-Capacitors:0.1UF-0603-25V-(+80/-20%) -> milador_SMD:CAP_CERAMIC-0603
- D1: device SparkFun-LED:LED-RED0603 -> milador_SMD:LED
- I2C: value JUMPER-SMT_3_2-NC_TRACE_SILK -> JUMPERS_JUMPER-SMT_3_2-NC_TRACE_SILK; device SparkFun-Jumpers:JUMPER-SMT_3_2-NC_TRACE_SILK -> milador_SMD:JUMPERS_JUMPER-SMT_3_2-NC_TRACE_SILK
- J1, J4: value QWIIC -> QWIIC_RIGHT_ANGLE; device SparkFun-Connectors:QWIIC_CONNECTORJS-1MM -> milador_SMD:QWIIC_CONNECTORSJS-1MM
- J2: device SparkFun-Connectors:CONN_01PTH_NO_SILK_YES_STOP -> milador:CONNECTORS_CONN_01PTH_NO_SILK_YES_STOP
- J3, J5: device SparkFun-Connectors:CONN_041X04_NO_SILK -> milador:CONNECTORS_CONN_041X04_NO_SILK
- R1, R2, R5, R6, R7, R8, R9: device SparkFun-Resistors:2.2KOHM-0603-1/10W-1% -> milador_SMD:RESISTOR-0603
- R3: device SparkFun-Resistors:10KOHM-0603-1/10W-1% -> milador_SMD:RESISTOR-0603
- R4: device SparkFun-Resistors:1KOHM-0603-1/10W-1% -> milador_SMD:RESISTOR-0603
- U1: device SparkFun-IC-Conversion:TCA9534U -> milador_SMD:TCA9534U
Other:
- note added: "By: Milad Hajihassan"
- note added: "Cut the I2C Jumpers to remove pullups from the I2C bus"
- note added: "LED"
- note added: "Pull-Ups"
- note added: "Visuals"
- note removed: "Cut the I2C Jumpers to remove these pullups from the I2C bus"
- note removed: "Developed By: Kevin Kuwata"
- note removed: "Modified By: Milad Hajihassan"
- note removed: "VCC: 1.65-5.5V"
- moved on the sheet: C1, D1, I2C, INT, PWR, U1

Commit message: Updated the design - Stable design
Connections:
- net GND: now also SW1.3, SW2.3
Changed lines of the file:
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@@
 <pinref part="SW2" gate="G$1" pin="1"/>
 <pinref part="GND12" gate="1" pin="GND"/>
-<wire x1="68.58" y1="175.26" x2="76.2" y2="175.26" width="0.1524" layer="91"/>
+<wire x1="68.58" y1="175.26" x2="71.12" y2="175.26" width="0.1524" layer="91"/>
+<pinref part="SW2" gate="G$1" pin="3"/>
+<wire x1="71.12" y1="175.26" x2="76.2" y2="175.26" width="0.1524" layer="91"/>
+<wire x1="68.58" y1="172.72" x2="71.12" y2="172.72" width="0.1524" layer="91"/>
+<wire x1="71.12" y1="172.72" x2="71.12" y2="175.26" width="0.1524" layer="91"/>
+<junction x="71.12" y="175.26"/>
 </segment>
 <segment>
 <pinref part="SW1" gate="G$1" pin="1"/>
 <pinref part="GND13" gate="1" pin="GND"/>
-<wire x1="119.38" y1="175.26" x2="124.46" y2="175.26" width="0.1524" layer="91"/>
+<wire x1="119.38" y1="175.26" x2="121.92" y2="175.26" width="0.1524" layer="91"/>
+<pinref part="SW1" gate="G$1" pin="3"/>
+<wire x1="121.92" y1="175.26" x2="124.46" y2="175.26" width="0.1524" layer="91"/>
+<wire x1="119.38" y1="172.72" x2="121.92" y2="172.72" width="0.1524" layer="91"/>
+<wire x1="121.92" y1="172.72" x2="121.92" y2="175.26" width="0.1524" layer="91"/>
+<junction x="121.92" y="175.26"/>
 </segment>
 <segment>
