File: Hardware/PCB/Eagle/Qwiic_Adaptive_Switch_Input.brd (EAGLE design)
At the start: 43.2 x 38.1 mm, 57 parts, among them J1 QWIIC_RIGHT_ANGLE, J4 QWIIC_RIGHT_ANGLE, SW1 CUI_SJ1-3513, SW2 CUI_SJ1-3513, U1 TCA9534

Commit message: Renamed the module
Parts:
- added U$27, U$28: MILADOR-SWITCH-NAME-SW-INPUT, milador:SWITCH-INPUT
- R5: value 10k -> 4.7k
- R6: value 10K -> 4.7K
- moved U$20 3.61 mm to (26.3, 22.0)
- moved U$19 3.43 mm to (27.0, 20.0)
- moved U$6 2.17 mm to (31.0, 18.5)
- moved U$16 1.88 mm to (33.0, 14.0)
Changed lines of the file:
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@@
 <setting verticaltext="up"/>
 </settings>
-<grid distance="0.005" unitdist="inch" unit="inch" style="lines" multiple="1" display="yes" altdistance="0.005" altunitdist="inch" altunit="inch"/>
+<grid distance="1.2" unitdist="mil" unit="mm" style="lines" multiple="1" display="yes" altdistance="0.005" altunitdist="inch" altunit="inch"/>
 <layers>
 <layer number="1" name="Top" color="4" fill="1" visible="yes" active="yes"/>
@@
 <layer number="199" name="Contour" color="7" fill="1" visible="no" active="no"/>
 <layer number="200" name="200bmp" color="1" fill="10" visible="yes" active="yes"/>
-<layer number="201" name="201bmp" color="1" fill="10" visible="yes" active="yes"/>
+<layer number="201" name="201bmp" color="2" fill="10" visible="yes" active="yes"/>
 <layer number="202" name="202bmp" color="3" fill="10" visible="no" active="no"/>
 <layer number="203" name="203bmp" color="4" fill="10" visible="no" active="no"/>
@@
 </layers>
 <board>
-<fusionsync huburn="a.cGVyc29uYWw6dWUyYWQxOTI2" projecturn="a.cGVyc29uYWw6dWUyYWQxOTI2IzIwMjEwMTA3MzY5MTI4NTU2" f3durn="urn:adsk.wipprod:dm.lineage:iqi4HTDMROu8o-H5T5Jb5A" pcbguid="" lastpulledtime="" lastsyncedchangeguid="" latestrevisionid="a4c49c8c-9ee0-401c-9360-ad30710fd072" lastsyncedrevisionid="a4c49c8c-9ee0-401c-9360-ad30710fd072" lastboardhashguid="7686bb73-5b86-c421-8fb9-e947596aed68" lastpushedtime="2021-06-23T00:17:49Z" linktopcb3d="true"/>
+<fusionsync huburn="a.cGVyc29uYWw6dWUyYWQxOTI2" projecturn="a.cGVyc29uYWw6dWUyYWQxOTI2IzIwMjEwMTA3MzY5MTI4NTU2" f3durn="urn:adsk.wipprod:dm.lineage:-B4RKxq_QYu-wduIUcvWIw" pcbguid="4d2b68f1-d6b2-48ec-84b6-8155f006826f" lastpulledtime="" lastsyncedchangeguid="" latestrevisionid="e58efc4d-1107-4ae5-a85b-ef9f61b83134" lastsyncedrevisionid="e58efc4d-1107-4ae5-a85b-ef9f61b83134" lastboardhashguid="d1f6887c-4ec4-a527-7b74-9df90bb43668" lastpushedtime="2021-09-05T00:20:39Z" linktopcb3d="true"/>
 <plain>
 <wire x1="0" y1="0" x2="0" y2="25.4" width="0.2032" layer="52"/>
@@
 <element name="SW1" library="MMC Eagle" library_urn="urn:adsk.eagle:library:13126479" package="CUI_SJ1-3513" package3d_urn="urn:adsk.eagle:package:25599488/3" value="CUI_SJ1-3513" x="13.462" y="36.322" smashed="yes" rot="R270">
 <attribute name="NAME" x="12.7" y="33.02" size="1.27" layer="21" ratio="15" rot="R270"/>
-<attribute name="VALUE" x="18.148359375" y="36.85506875" size="0.6096" layer="27" rot="R270" align="top-left"/>
 </element>
 <element name="J5" library="milador" library_urn="urn:adsk.eagle:library:12595918" package="CONNECTORS_1X04_NO_SILK" package3d_urn="urn:adsk.eagle:package:29222251/2" value="" x="41.91" y="6.35" smashed="yes" rot="R90">
@@
 <element name="U$2" library="buzzard_labels (44)" package="GND4" value="" x="36.83" y="6.35" smashed="yes"/>
 <element name="U$4" library="buzzard_labels (44)" package="3V33" value="" x="41.3512" y="8.89" smashed="yes" rot="MR0"/>
-<element name="R5" library="milador_SMD" library_urn="urn:adsk.eagle:library:27847482" package="0603" package3d_urn="urn:adsk.eagle:package:29222124/2" value="10k" x="17.78" y="22.098" smashed="yes">
+<element name="R5" library="milador_SMD" library_urn="urn:adsk.eagle:library:27847482" package="0603" package3d_urn="urn:adsk.eagle:package:29222124/2" value="4.7k" x="17.78" y="22.098" smashed="yes">
 <attribute name="NAME" x="17.78" y="21.209" size="0.8128" layer="21" font="vector" ratio="15" rot="R180" align="bottom-center"/>
 <attribute name="VALUE" x="17.907" y="23.495" size="0.6096" layer="27" font="vector" ratio="20" align="top-center"/>
 </element>
-<element name="R6" library="milador_SMD" library_urn="urn:adsk.eagle:library:27847482" package="0603" package3d_urn="urn:adsk.eagle:package:29222124/2" value="10K" x="22.86" y="22.098" smashed="yes" rot="R180">
+<element name="R6" library="milador_SMD" library_urn="urn:adsk.eagle:library:27847482" package="0603" package3d_urn="urn:adsk.eagle:package:29222124/2" value="4.7K" x="22.86" y="22.098" smashed="yes" rot="R180">
 <attribute name="NAME" x="22.86" y="21.209" size="0.8128" layer="21" font="vector" ratio="15" rot="R180" align="bottom-center"/>
 <attribute name="VALUE" x="22.86" y="22.86" size="0.6096" layer="27" font="vector" ratio="20" rot="R180" align="top-center"/>
@@
 <attribute name="VALUE" x="27.94" y="12.827" size="0.6096" layer="28" font="vector" ratio="20" rot="MR180" align="top-center"/>
 </element>
-<element name="U$6" library="milador" library_urn="urn:adsk.eagle:library:12595918" package="MILADOR_LOGO1" package3d_urn="urn:adsk.eagle:package:28431737/1" value="MILADOR-LOGO-" x="31.7754" y="16.4719" smashed="yes" rot="R90"/>
+<element name="U$6" library="milador" library_urn="urn:adsk.eagle:library:12595918" package="MILADOR_LOGO1" package3d_urn="urn:adsk.eagle:package:28431737/1" value="MILADOR-LOGO-" x="31" y="18.5" smashed="yes" rot="R90"/>
 <element name="U$8" library="buzzard_labels (44)" package="3V33" value="" x="36.83" y="8.89" smashed="yes"/>
 <element name="U$14" library="buzzard_labels (44)" package="GND4" value="" x="36.83" y="6.4008" smashed="yes" rot="MR180"/>
-<element name="U$16" library="milador" library_urn="urn:adsk.eagle:library:12595918" package="MILADOR_QWIIC_SWITCH" package3d_urn="urn:adsk.eagle:package:29091844/1" value="" x="33.8455" y="12.319" smashed="yes" rot="R90"/>
+<element name="U$16" library="milador" library_urn="urn:adsk.eagle:library:12595918" package="MILADOR_QWIIC_SWITCH" package3d_urn="urn:adsk.eagle:package:29091844/1" value="" x="33" y="14" smashed="yes" rot="R90"/>
 <element name="U$17" library="milador" library_urn="urn:adsk.eagle:library:12595918" package="SWITCH-SW1" package3d_urn="urn:adsk.eagle:package:29091877/1" value="MILADOR-SWITCH-NAME-SW1" x="13.9065" y="32.9438" smashed="yes" rot="MR0"/>
 <element name="U$18" library="milador" library_urn="urn:adsk.eagle:library:12595918" package="SWITCH-SW2" package3d_urn="urn:adsk.eagle:package:29091878/1" value="MILADOR-SWITCH-NAME-SW2" x="30.1625" y="32.9438" smashed="yes" rot="MR0"/>
-<element name="U$19" library="milador" library_urn="urn:adsk.eagle:library:12595918" package="MILADOR_QWIIC_SWITCH" package3d_urn="urn:adsk.eagle:package:29091844/1" value="" x="26.797" y="16.5735" smashed="yes" rot="MR0"/>
-<element name="U$20" library="milador" library_urn="urn:adsk.eagle:library:12595918" package="MILADOR_LOGO1" package3d_urn="urn:adsk.eagle:package:28431737/1" value="MILADOR-LOGO-" x="26.3144" y="18.3896" smashed="yes" rot="MR0"/>
+<element name="U$19" library="milador" library_urn="urn:adsk.eagle:library:12595918" package="MILADOR_QWIIC_SWITCH" package3d_urn="urn:adsk.eagle:package:29091844/1" value="" x="27" y="20" smashed="yes" rot="MR0"/>
+<element name="U$20" library="milador" library_urn="urn:adsk.eagle:library:12595918" package="MILADOR_LOGO1" package3d_urn="urn:adsk.eagle:package:28431737/1" value="MILADOR-LOGO-" x="26.3144" y="22" smashed="yes" rot="MR0"/>
+<element name="U$27" library="milador" library_urn="urn:adsk.eagle:library:12595918" package="SWITCH-INPUT" package3d_urn="urn:adsk.eagle:package:30678307/1" value="MILADOR-SWITCH-NAME-SW-INPUT" x="35.5" y="21.2" smashed="yes" rot="R90"/>
+<element name="U$28" library="milador" library_urn="urn:adsk.eagle:library:12595918" package="SWITCH-INPUT" package3d_urn="urn:adsk.eagle:package:30678307/1" value="MILADOR-SWITCH-NAME-SW-INPUT" x="19.8" y="17.5" smashed="yes" rot="MR0"/>
 </elements>
 <signals>
