File: Hardware/PCB/Eagle/Qwiic_Adaptive_Switch_Input.sch (EAGLE design)
At the start: 32 parts, among them J1 QWIIC_RIGHT_ANGLE, J4 QWIIC_RIGHT_ANGLE, SW1 CUI_SJ1-3513, SW2 CUI_SJ1-3513, U1 TCA9534

Commit message: Renamed the module
Parts:
- added U$27, U$28: MILADOR-SWITCH-NAME-SW-INPUT, milador:MILADOR-SWITCH-NAME-SW-INPUT
- R5: value 10k -> 4.7k
- R6: value 10K -> 4.7K
Changed lines of the file:
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@@
 <part name="SUPPLY10" library="SparkFun-PowerSymbols" deviceset="3.3V" device=""/>
 <part name="FRAME1" library="frames" library_urn="urn:adsk.eagle:library:229" deviceset="TABL_L" device=""/>
-<part name="R5" library="milador_SMD" library_urn="urn:adsk.eagle:library:27847482" deviceset="RESISTOR-" device="0603" package3d_urn="urn:adsk.eagle:package:29222124/2" value="10k"/>
+<part name="R5" library="milador_SMD" library_urn="urn:adsk.eagle:library:27847482" deviceset="RESISTOR-" device="0603" package3d_urn="urn:adsk.eagle:package:29222124/2" value="4.7k"/>
 <part name="SUPPLY11" library="SparkFun-PowerSymbols" deviceset="3.3V" device=""/>
-<part name="R6" library="milador_SMD" library_urn="urn:adsk.eagle:library:27847482" deviceset="RESISTOR-" device="0603" package3d_urn="urn:adsk.eagle:package:29222124/2" value="10K"/>
+<part name="R6" library="milador_SMD" library_urn="urn:adsk.eagle:library:27847482" deviceset="RESISTOR-" device="0603" package3d_urn="urn:adsk.eagle:package:29222124/2" value="4.7K"/>
 <part name="SUPPLY15" library="SparkFun-PowerSymbols" deviceset="3.3V" device=""/>
 <part name="ADR2" library="milador_SMD" library_urn="urn:adsk.eagle:library:27847482" deviceset="JUMPERS-SMT_2_NC_TRACE" device="_SILK" package3d_urn="urn:adsk.eagle:package:29222215/1" value="JUMPERS-SMT_2_NC_TRACE_SILK"/>
@@
 <part name="U$17" library="milador" library_urn="urn:adsk.eagle:library:12595918" deviceset="MILADOR-SWITCH-NAME-" device="SW1" package3d_urn="urn:adsk.eagle:package:29091877/1"/>
 <part name="U$18" library="milador" library_urn="urn:adsk.eagle:library:12595918" deviceset="MILADOR-SWITCH-NAME-" device="SW2" package3d_urn="urn:adsk.eagle:package:29091878/1"/>
+<part name="U$27" library="milador" library_urn="urn:adsk.eagle:library:12595918" deviceset="MILADOR-SWITCH-NAME-" device="SW-INPUT" package3d_urn="urn:adsk.eagle:package:30678307/1"/>
+<part name="U$28" library="milador" library_urn="urn:adsk.eagle:library:12595918" deviceset="MILADOR-SWITCH-NAME-" device="SW-INPUT" package3d_urn="urn:adsk.eagle:package:30678307/1"/>
 </parts>
 <sheets>
@@
 <instance part="U$17" gate="G$1" x="142.24" y="12.7" smashed="yes"/>
 <instance part="U$18" gate="G$1" x="157.48" y="12.7" smashed="yes"/>
+<instance part="U$27" gate="G$1" x="142.24" y="0" smashed="yes"/>
+<instance part="U$28" gate="G$1" x="157.48" y="0" smashed="yes"/>
 </instances>
 <busses>
